File: Electronics/CitationX_cockpit/copilot_APU.sch (KiCad schematic (older format))
At the start: 0 parts

Commit message: Electronics - Working on APUs
Parts:
- added C? (x3): 0.1u, symbol Device:C_Small
- added J? (x3): Screw_Terminal_01x10, symbol Connector:Screw_Terminal_01x10
- added RN?: R_Network08, Resistor_THT:R_Array_SIP9, symbol Device:R_Network08
- added U?: ProMicro, symbol promicro:ProMicro
- added U? (x2): 74HC4051, symbol 74xx:74HC4051
- added U?: 74HC165, symbol pkl_misc:74HC165
Connections:
- new net +3V3: C?.1, C?.1, C?.1, RN?.1 (common), U?.16 (VCC), U?.16 (VCC), U?.16 (VCC)
- new net +5V: J?.10 (Pin_10), J?.7 (Pin_7), J?.8 (Pin_8), J?.9 (Pin_9), U?.21 (VCC)
- new net 7SEG_CLK: U?.11 (B4), U?.3 (A)
- new net 7SEG_DIO: U?.10 (E6), U?.3 (A)
- new net APU_START: J?.6 (Pin_6), RN?.4 (R3), U?.4 (D5)
- new net APU_START_DIS: J?.5 (Pin_5), RN?.5 (R4), U?.3 (D4)
- new net APU_STOP: J?.7 (Pin_7), RN?.3 (R2), U?.5 (D6)
- new net BLEED_MAX: J?.1 (Pin_1), RN?.9 (R8), U?.11 (D0)
- new net BLEED_OFF: J?.2 (Pin_2), RN?.8 (R7), U?.12 (D1)
- new net CLK: U?.15 (B3), U?.2 (CLK)
- new net CLK0: J?.1 (Pin_1), U?.13 (A0)
- new net CLK1: J?.3 (Pin_3), U?.14 (A1)
- new net CLK2: J?.5 (Pin_5), U?.15 (A2)
- new net CLK3: J?.7 (Pin_7), U?.12 (A3)
- new net CLK4: J?.9 (Pin_9), U?.1 (A4)
- new net DIO0: J?.2 (Pin_2), U?.13 (A0)
- new net DIO1: J?.4 (Pin_4), U?.14 (A1)
- new net DIO2: J?.6 (Pin_6), U?.15 (A2)
- new net DIO3: J?.8 (Pin_8), U?.12 (A3)
- new net DIO4: J?.10 (Pin_10), U?.1 (A4)
- new net E: U?.12 (B5), U?.6 (~E), U?.6 (~E)
- new net GEN_ON: J?.3 (Pin_3), RN?.7 (R6), U?.13 (D2)
- new net GEN_RST: J?.4 (Pin_4), RN?.6 (R5), U?.14 (D3)
- new net GND: C?.2, C?.2, C?.2, J?.1 (Pin_1), J?.2 (Pin_2), J?.3 (Pin_3), J?.4 (Pin_4), J?.5 (Pin_5), U?.10 (SER), U?.15 (CLK_INH), U?.23 (GND), U?.7 (VEE), U?.7 (VEE), U?.8 (GND), U?.8 (GND), U?.8 (GND)
- new net ISR_LATCH: U?.1 (SH/~LD), U?.14 (B2)
- new net ISR_OUT: U?.13 (B6), U?.9 (QH)
- new net L0: U?.11 (S0), U?.11 (S0), U?.7 (D4)
- new net L1: U?.10 (S1), U?.10 (S1), U?.8 (C6)
- new net L2: U?.9 (D7), U?.9 (S2), U?.9 (S2)
- new net MAP_LIGHT: U?.18 (F6)
- new net MASTER_ON: U?.16 (B1)
- new net PB_TEST: J?.8 (Pin_8), RN?.2 (R1), U?.6 (D7)
- new net POT_X1: U?.17 (F7)
- new net SCL: U?.5 (SCL)
- new net SDA: U?.6 (SDA)
- no-connect marks 0 -> 15
Other:
- note added: "Connectors for 7x 7-seg"
- note added: "The ProMicro will receive the values to be displayed on \nthe 7-segments via I2C. It will then take care of the diaplays."

Commit message: Electronics - Misc. works
Continued (and checked board). All connections are probably OK.
Fixed hierarchical pins in APUs (affects all schematics)
Numbered elements for testing schematics
Parts:
- gave numbers to parts that had none: 11
Connections:
- net GND: no longer U57.10 (SER)
- new net ISR_IN: U57.10 (SER)
- no-connect marks 15 -> 17

Commit message: Electronics - Copied pilot_APU in copilot_APU
Parts:
- removed C64, C65, C66: 0.1u, symbol Device:C_Small
- removed J40, J41, J42: Screw_Terminal_01x10, symbol Connector:Screw_Terminal_01x10
- removed RN28: R_Network08, Resistor_THT:R_Array_SIP9, symbol Device:R_Network08
- removed U57: 74HC165, symbol pkl_misc:74HC165
- removed U58: ProMicro, symbol promicro:ProMicro
- removed U59, U60: 74HC4051, symbol 74xx:74HC4051
- added C? (x3): 0.1u, symbol Device:C_Small
- added J? (x3): Screw_Terminal_01x10, symbol Connector:Screw_Terminal_01x10
- added J?: Conn_02x08_Odd_Even, symbol Connector_Generic:Conn_02x08_Odd_Even
- added RN?: R_Network08, Resistor_THT:R_Array_SIP9, symbol Device:R_Network08
- added U?: ProMicro, symbol promicro:ProMicro
- added U? (x2): 74HC4051, symbol 74xx:74HC4051
- added U?: 74HC165, symbol pkl_misc:74HC165
Connections:
- net labels added: RST, RX, TX
- net labels removed: ISR_IN
- wire segments 28 -> 26
- no-connect marks 17 -> 14
Other:
- note added: "Connectors for 7x 7-seg and OLED\n"
- note added: "RST can be used to restart the Pro Micro.\nThis pin is pulled high by a 10k resistor on the board, \nand is active-low, so it must be connected to ground to initiate a reset.\nThe Pro Micro will remain "off" until the reset line is pulled back to high."
- note added: "SCL and SDA are used for an OLED\n"
- note added: "This board will be separated from the rest.\nIw ill communicate with the master using USART (TTL level, no need for MAX232)"
- note removed: "Connectors for 7x 7-seg"
- note removed: "The ProMicro will receive the values to be displayed on \nthe 7-segments via I2C. It will then take care of the diaplays."
