File: Electronics/CitationX_cockpit/CitationX_cockpit.sch (KiCad schematic (older format))
At the start: 44 parts, among them J1 Raspberry_Pi_2_3, U1 ESP32-WROOM-32

Commit message: Electronics - Working on copilot side and APU
Changed lines of the file:
@@
 F0 "copilot" 50
 F1 "copilot.sch" 50
+F2 "ISR_IN" I L 4500 6650 50
+F3 "ISR_OUT" O R 5350 6650 50
+F4 "OSR_IN" I L 4500 6750 50
+F5 "OSR_OUT" O R 5350 6750 50
 $EndSheet
 $Sheet

Commit message: Electronics - Misc. works
Continued (and checked board). All connections are probably OK.
Fixed hierarchical pins in APUs (affects all schematics)
Numbered elements for testing schematics
Parts:
- removed C? (x4): 0.1u, symbol Device:C_Small
- removed U? (x4): PCF8575, IPC7351-Nominal:SOP65P775X200-24, symbol NXP:PCF8575
- gave numbers to parts that had none: 34

Commit message: Electronics - Misc works
Changed lines of the file:
@@
 F1 "board.sch" 50
 F2 "ISR_IN" I L 3100 5850 50
-F3 "ISR_LATCH" I L 3100 5950 50
-F4 "CLK" I L 3100 5600 50
 F5 "ISR_OUT" O R 5650 5850 50
 F6 "OSR_IN" I L 3100 6100 50
@@
 F0 "autopilot" 50
 F1 "autopilot.sch" 50
+F2 "ISR_IN" I L 3800 5200 50
+F3 "OSR_IN" I L 3800 5300 50
+F4 "OSR_OUT" O R 4950 5300 50
+F5 "ISR_OUT" O R 4950 5200 50
 $EndSheet
 $Comp

Commit message: Electronics - Misc works
Parts:
- removed C10, C11, C12, C13, C14, C15, C16, C17, C8: 100u, symbol Device:CP_Small
- removed C5, C7: 100n, symbol Device:C_Small
- removed C6, C9: 0.1u, symbol Device:C_Small
- removed D1: LED_Small, symbol Device:LED_Small
- removed J1: Raspberry_Pi_2_3, symbol Connector:Raspberry_Pi_2_3
- removed J2, J3, J4, J5, J6, J7, J8, J9: Screw_Terminal_01x03, symbol Connector:Screw_Terminal_01x03
- removed R1: 68, symbol Device:R_Small
- removed R2, R3, R4, R5, R6, R7, R8, R9: 470, symbol Device:R
- removed U1: ESP32-WROOM-32, RF_Module:ESP32-WROOM-32, symbol RF_Module:ESP32-WROOM-32
- removed U6: 74HC4051, symbol 74xx:74HC4051
- removed U7: LD1117S33TR_SOT223, Package_TO_SOT_SMD:SOT-223-3_TabPin2, symbol Regulator_Linear:LD1117S33TR_SOT223
- removed U8: 74HC595, symbol 74xx:74HC595
Other:
- note removed: "3.3V generation\ncheck if 800 mA is enough"

Commit message: Fixed the previous commit, CitationX_cockpit.sch got emptied
Parts:
- added C10, C11, C12, C13, C14, C15, C16, C17, C8: 100u, symbol Device:CP_Small
- added C5, C7: 100n, symbol Device:C_Small
- added C6, C9: 0.1u, symbol Device:C_Small
- added D1: LED_Small, symbol Device:LED_Small
- added J1: Raspberry_Pi_2_3, symbol Connector:Raspberry_Pi_2_3
- added J2, J3, J4, J5, J6, J7, J8, J9: Screw_Terminal_01x03, symbol Connector:Screw_Terminal_01x03
- added R1: 68, symbol Device:R_Small
- added R2, R3, R4, R5, R6, R7, R8, R9: 470, symbol Device:R
- added U1: ESP32-WROOM-32, RF_Module:ESP32-WROOM-32, symbol RF_Module:ESP32-WROOM-32
- added U6: 74HC4051, symbol 74xx:74HC4051
- added U7: LD1117S33TR_SOT223, Package_TO_SOT_SMD:SOT-223-3_TabPin2, symbol Regulator_Linear:LD1117S33TR_SOT223
- added U8: 74HC595, symbol 74xx:74HC595
Connections:
- new net: J2.3 (Pin_3), R2.2
- new net: J3.3 (Pin_3), R3.2
- new net: J4.3 (Pin_3), R4.2
- new net: J5.3 (Pin_3), R5.2
- new net: J6.3 (Pin_3), R6.2
- new net: J7.3 (Pin_3), R7.2
- new net: J8.3 (Pin_3), R8.2
- new net: J9.3 (Pin_3), R9.2
- new net: C5.2, C7.2, C8.2, R1.2, U7.1 (GND)
- new net: D1.1 (K), R1.1
- new net +3V3: C6.1, C7.1, C8.1, C9.1, D1.2 (A), U6.16 (VCC), U7.2 (VO), U8.10 (~SRCLR), U8.16 (VCC)
- new net +5V: C10.1, C11.1, C12.1, C13.1, C14.1, C15.1, C16.1, C17.1, C5.1, J2.1 (Pin_1), J3.1 (Pin_1), J4.1 (Pin_1), J5.1 (Pin_1), J6.1 (Pin_1), J7.1 (Pin_1), J8.1 (Pin_1), J9.1 (Pin_1), U7.3 (VI)
- new net CLK: U8.11 (SRCLK)
- new net GND: C10.2, C11.2, C12.2, C13.2, C14.2, C15.2, C16.2, C17.2, C6.2, C9.2, J2.2 (Pin_2), J3.2 (Pin_2), J4.2 (Pin_2), J5.2 (Pin_2), J6.2 (Pin_2), J7.2 (Pin_2), J8.2 (Pin_2), J9.2 (Pin_2), U1.1 (GND), U1.15 (GND), U1.38 (GND), U6.7 (VEE), U6.8 (GND), U8.13 (~OE), U8.8 (GND)
- new net LIGHT: U6.3 (A)
- new net LIGHT_AP: R4.1, U6.15 (A2)
- new net LIGHT_APU: R6.1, U6.1 (A4)
- new net LIGHT_CENTER: R5.1, U6.12 (A3)
- new net LIGHT_COPILOT: R3.1, U6.14 (A1)
- new net LIGHT_E: U6.6 (~E)
- new net LIGHT_PILOT: R2.1, U6.13 (A0)
- new net LIGHT_X1: R7.1, U6.5 (A5)
- new net LIGHT_X2: R8.1, U6.2 (A6)
- new net LIGHT_X3: R9.1, U6.4 (A7)
- new net OSR_IN: U8.14 (SER)
- new net OSR_LATCH: U8.12 (RCLK)
- new net OSR_OUT: U8.9 (QH')
- new net OSR_X1: U8.5 (QF)
- new net OSR_X2: U8.6 (QG)
- new net OSR_X3: U8.7 (QH)
- new net P_APU_ADC_E: U8.3 (QD)
- new net P_SIDE_ADC_E: U8.4 (QE)
- new net RX: J1.10 (GPIO15/RXD), U1.35 (TXD0/IO1)
- new net S0: U6.11 (S0), U8.15 (QA)
- new net S1: U6.10 (S1), U8.1 (QB)
- new net S2: U6.9 (S2), U8.2 (QC)
- new net SCL: J1.5 (SCL/GPIO3), U1.22 (SDI/SD1)
- new net SDA: J1.3 (SDA/GPIO2), U1.21 (SDO/SD0)
- new net TX: J1.8 (GPIO14/TXD), U1.34 (RXD0/IO3)
Other:
- note added: "3.3V generation\ncheck if 800 mA is enough"

Commit message: Electronics - Misc works
Changed lines of the file:
@@
 EESchema Schematic File Version 4
 LIBS:CitationX_cockpit-cache
-EELAYER 30 0
+EELAYER 26 0
 EELAYER END
 $Descr A3 11693 16535 portrait
@@
 F4 "OSR_IN" I L 3100 6100 50
 F5 "OSR_OUT" O R 5650 6100 50
-F6 "OSR_LATCH" I L 3100 6200 50
 $EndSheet
 $Comp
@@
 LIGHT_E
 $Sheet
-S 4100 7650 650  850
+S 4000 7650 850  850
 U 5DBF6FEB
 F0 "pedestral" 50
 F1 "pedestral.sch" 50
+F2 "ADC_E" I L 4000 8400 50
+F3 "ISR_IN" I L 4000 7750 50
+F4 "OSR_IN" I L 4000 7850 50
+F5 "OSR_OUT" I R 4850 7850 50
+F6 "ISR_OUT" I R 4850 7750 50
 $EndSheet
 $Sheet

Commit message: Electronics - Moved library to root of Electronics
Changed lines of the file:
@@
 $Descr A3 11693 16535 portrait
 encoding utf-8
-Sheet 1 10
+Sheet 1 8
 Title ""
 Date ""
@@
 $EndSheet
 $Sheet
-S 550  5950 900  1400
-U 5DC174D6
-F0 "pilot_APU" 50
-F1 "pilot_APU.sch" 50
-F2 "ISR_LATCH" I L 550 6300 50
-F3 "CLK" I L 550 6050 50
-F4 "ISR_OUT" O R 1450 6150 50
-F5 "ISR_IN" I L 550 6200 50
-$EndSheet
-$Sheet
 S 4500 6550 850  550
 U 5DC2EEA6
@@
 $EndSheet
 $Sheet
-S 7650 5950 900  1400
-U 5DC313C6
-F0 "copilot_APU" 50
-F1 "copilot_APU.sch" 50
-F2 "ISR_LATCH" I L 7650 6300 50
-F3 "ISR_OUT" O R 8550 6150 50
-F4 "ISR_IN" I L 7650 6200 50
-F5 "CLK" I L 7650 6050 50
-$EndSheet
-$Sheet
