File: Electronics/CitationX_cockpit/copilot_side.sch (KiCad schematic (older format))
At the start: 18 parts

Commit message: Electronics - Working on copilot side and APU
Connections:
- net BP_ADC_REV renamed PB_ADC_REV
- net BP_CABIN renamed PB_CABIN
- net BP_EMER renamed PB_EMER
- net BP_HF_1 renamed PB_HF_1
- net BP_IRV_REV renamed PB_IRS_REV
- net BP_MUTE renamed PB_MUTE
- net PB_DG_TEST renamed PB_SG_TEST

Commit message: Electronics - Misc. works
Continued (and checked board). All connections are probably OK.
Fixed hierarchical pins in APUs (affects all schematics)
Numbered elements for testing schematics
Parts:
- gave numbers to parts that had none: 18

Commit message: Electronics - Misc works
Parts:
- added U?: ULN2803A, symbol Transistor_Array:ULN2803A
Connections:
- net CABIN: now also U?.16 (O3); no longer U56.3 (QD)
- net COM_1: now also U?.10 (COM); no longer U56.15 (QA)
- net COM_2: now also U?.18 (O1); no longer U56.1 (QB)
- net EMER: now also U?.15 (O4); no longer U56.4 (QE)
- net GND: now also U?.9 (GND)
- net HF_1: now also U?.17 (O2); no longer U56.2 (QC)
- net at U56.5 (QF): now also U?.6 (I6)
- net at U56.6 (QG): now also U?.7 (I7)
- net at U56.7 (QH): now also U?.8 (I8)
- new net: U56.1 (QB), U?.2 (I2)
- new net: U56.15 (QA), U?.1 (I1)
- new net: U56.2 (QC), U?.3 (I3)
- new net: U56.3 (QD), U?.4 (I4)
- new net: U56.4 (QE), U?.5 (I5)
Other:
- moved on the sheet: C63, U55
Changed lines of the file:
@@
 EESchema Schematic File Version 4
 LIBS:CitationX_cockpit-cache
-EELAYER 30 0
+EELAYER 26 0
 EELAYER END
 $Descr A4 8268 11693 portrait
@@
 L 74xx:74HC4051 U?
 U 1 1 5DC023F6
-P 6100 4850
+P 6100 5000
 AR Path="/5DB5DCD1/5DC023F6" Ref="U?"  Part="1"
 AR Path="/5DC174D4/5DC023F6" Ref="U?"  Part="1"
 AR Path="/5DC31399/5DC023F6" Ref="U55"  Part="1"
-F 0 "U55" H 6150 5528 50  0000 C CNN
-F 1 "74HC4051" H 6150 5437 50  0000 C CNN
-F 2 "" H 6100 4450 50  0001 C CNN
-F 3 "http://www.ti.com/lit/ds/symlink/cd74hc4051.pdf" H 6100 4450 50  0001 C CNN
-	1    6100 4850
+F 0 "U55" H 6150 5678 50  0000 C CNN
+F 1 "74HC4051" H 6150 5587 50  0000 C CNN
+F 2 "" H 6100 4600 50  0001 C CNN
+F 3 "http://www.ti.com/lit/ds/symlink/cd74hc4051.pdf" H 6100 4600 50  0001 C CNN
+	1    6100 5000
 	1    0    0    -1
 $EndComp
@@
 COM1_LSPK
 Wire Wire Line
-	6100 5450 6150 5450
+	6100 5600 6150 5600
 $Comp
 L power:GND #PWR?
 U 1 1 5DC02402
-P 6150 5450
+P 6150 5600
 AR Path="/5DB5DCD1/5DC02402" Ref="#PWR?"  Part="1"
 AR Path="/5DC174D4/5DC02402" Ref="#PWR?"  Part="1"
 AR Path="/5DC31399/5DC02402" Ref="#PWR0377"  Part="1"
-F 0 "#PWR0377" H 6150 5200 50  0001 C CNN
-F 1 "GND" H 6155 5277 50  0000 C CNN
-F 2 "" H 6150 5450 50  0001 C CNN
-F 3 "" H 6150 5450 50  0001 C CNN
-	1    6150 5450
-	1    0    0    -1
-$EndComp
-Connection ~ 6150 5450
-Wire Wire Line
-	6150 5450 6200 5450
+F 0 "#PWR0377" H 6150 5350 50  0001 C CNN
+F 1 "GND" H 6155 5427 50  0000 C CNN
+F 2 "" H 6150 5600 50  0001 C CNN
+F 3 "" H 6150 5600 50  0001 C CNN
+	1    6150 5600
+	1    0    0    -1
+$EndComp
+Connection ~ 6150 5600
+Wire Wire Line
+	6150 5600 6200 5600
 $Comp
 L Device:C_Small C?
 U 1 1 5DC0240A
-P 6550 4350
+P 6550 4500
 AR Path="/5DB5DCD1/5DC0240A" Ref="C?"  Part="1"
 AR Path="/5DC174D4/5DC0240A" Ref="C?"  Part="1"
 AR Path="/5DC31399/5DC0240A" Ref="C63"  Part="1"
-F 0 "C63" V 6779 4350 50  0000 C CNN
-F 1 "0.1u" V 6688 4350 50  0000 C CNN
-F 2 "" H 6550 4350 50  0001 C CNN
-F 3 "~" H 6550 4350 50  0001 C CNN
-	1    6550 4350
-	0    -1   -1   0
-$EndComp
-Wire Wire Line
-	6100 4350 6450 4350
+F 0 "C63" V 6779 4500 50  0000 C CNN
+F 1 "0.1u" V 6688 4500 50  0000 C CNN
+F 2 "" H 6550 4500 50  0001 C CNN
+F 3 "~" H 6550 4500 50  0001 C CNN
+	1    6550 4500
+	0    -1   -1   0
+$EndComp
+Wire Wire Line
+	6100 4500 6450 4500
 $Comp
 L power:GND #PWR?
 U 1 1 5DC02412
-P 6650 4350
+P 6650 4500
 AR Path="/5DB5DCD1/5DC02412" Ref="#PWR?"  Part="1"
 AR Path="/5DC174D4/5DC02412" Ref="#PWR?"  Part="1"
 AR Path="/5DC31399/5DC02412" Ref="#PWR0378"  Part="1"
-F 0 "#PWR0378" H 6650 4100 50  0001 C CNN
-F 1 "GND" V 6655 4222 50  0000 R CNN
-F 2 "" H 6650 4350 50  0001 C CNN
-F 3 "" H 6650 4350 50  0001 C CNN
-	1    6650 4350
+F 0 "#PWR0378" H 6650 4250 50  0001 C CNN
+F 1 "GND" V 6655 4372 50  0000 R CNN
+F 2 "" H 6650 4500 50  0001 C CNN
+F 3 "" H 6650 4500 50  0001 C CNN
+	1    6650 4500
 	0    -1   -1   0
 $EndComp
@@
 L power:+3.3V #PWR?
 U 1 1 5DC02418
-P 5900 4350
+P 5900 4500
 AR Path="/5DB5DCD1/5DC02418" Ref="#PWR?"  Part="1"
 AR Path="/5DC174D4/5DC02418" Ref="#PWR?"  Part="1"
 AR Path="/5DC31399/5DC02418" Ref="#PWR0379"  Part="1"
-F 0 "#PWR0379" H 5900 4200 50  0001 C CNN
-F 1 "+3.3V" V 5915 4478 50  0000 L CNN
-F 2 "" H 5900 4350 50  0001 C CNN
-F 3 "" H 5900 4350 50  0001 C CNN
-	1    5900 4350
-	0    -1   -1   0
-$EndComp
-Connection ~ 6100 4350
-Wire Wire Line
-	5900 4350 6100 4350
-Text HLabel 5800 4550 0    50   Output ~ 0
+F 0 "#PWR0379" H 5900 4350 50  0001 C CNN
+F 1 "+3.3V" V 5915 4628 50  0000 L CNN
+F 2 "" H 5900 4500 50  0001 C CNN
+F 3 "" H 5900 4500 50  0001 C CNN
+	1    5900 4500
+	0    -1   -1   0
+$EndComp
+Connection ~ 6100 4500
+Wire Wire Line
+	5900 4500 6100 4500
+Text HLabel 5800 4700 0    50   Output ~ 0
 ADC
-Text HLabel 5800 5150 0    50   Input ~ 0
+Text HLabel 5800 5300 0    50   Input ~ 0
 ADC_E_1
 Text Label 6700 2600 0    50   ~ 0
@@
 Text Label 6700 3800 0    50   ~ 0
 SPKR
-Text Label 6500 4550 0    50   ~ 0
+Text Label 6500 4700 0    50   ~ 0
 MLS_1
-Text Label 6500 4650 0    50   ~ 0
+Text Label 6500 4800 0    50   ~ 0
 MLS_2
-Text Label 6500 4750 0    50   ~ 0
+Text Label 6500 4900 0    50   ~ 0
 MKR
-Text Label 6500 4850 0    50   ~ 0
+Text Label 6500 5000 0    50   ~ 0
 HDPH
-Text GLabel 5800 4850 0    50   Input ~ 0
+Text GLabel 5800 5000 0    50   Input ~ 0
 A1
-Text GLabel 5800 4950 0    50   Input ~ 0
+Text GLabel 5800 5100 0    50   Input ~ 0
 A2
-Text GLabel 5800 4750 0    50   Input ~ 0
+Text GLabel 5800 4900 0    50   Input ~ 0
 A0
 $Comp
@@
 	1    0    0    -1
 $EndComp
-Text HLabel 6500 7450 2    50   Output ~ 0
+Text HLabel 6500 7450 3    50   Output ~ 0
 OSR_OUT
 $Comp
@@
 Text GLabel 5700 6750 0    50   Input ~ 0
 CLK
-Text Label 6500 6550 0    50   ~ 0
+Text Label 7300 6450 0    50   ~ 0
 COM_1
-Text Label 6500 6650 0    50   ~ 0
+Text Label 7300 6550 0    50   ~ 0
 COM_2
-Text Label 6500 6750 0    50   ~ 0
+Text Label 7300 6650 0    50   ~ 0
 HF_1
-Text Label 6500 6850 0    50   ~ 0
+Text Label 7300 6750 0    50   ~ 0
 CABIN
-Text Label 6500 6950 0    50   ~ 0
+Text Label 7300 6850 0    50   ~ 0
 EMER
+$Comp
+L Transistor_Array:ULN2803A U?
+U 1 1 5DEA06A1
+P 6900 6750
+AR Path="/5DBF6FEB/5DEA06A1" Ref="U?"  Part="1"
+AR Path="/5DC33C09/5DEA06A1" Ref="U?"  Part="1"
+AR Path="/5DC31399/5DEA06A1" Ref="U?"  Part="1"
+F 0 "U?" H 6900 7317 50  0000 C CNN
+F 1 "ULN2803A" H 6900 7226 50  0000 C CNN
+F 2 "" H 6950 6100 50  0001 L CNN
+F 3 "http://www.ti.com/lit/ds/symlink/uln2803a.pdf" H 7000 6550 50  0001 C CNN
+	1    6900 6750
+	1    0    0    -1
+$EndComp
+$Comp
+L power:GND #PWR?
+U 1 1 5DEA6F8F
+P 6900 7450
+AR Path="/5DB5DCD1/5DEA6F8F" Ref="#PWR?"  Part="1"
+AR Path="/5DC174D4/5DEA6F8F" Ref="#PWR?"  Part="1"
+AR Path="/5DC31399/5DEA6F8F" Ref="#PWR?"  Part="1"
+F 0 "#PWR?" H 6900 7200 50  0001 C CNN
+F 1 "GND" H 6905 7277 50  0000 C CNN
+F 2 "" H 6900 7450 50  0001 C CNN
+F 3 "" H 6900 7450 50  0001 C CNN
+	1    6900 7450
+	1    0    0    -1
+$EndComp
 $EndSCHEMATC
