File: Electronics/CitationX_cockpit/pedestral.sch (KiCad schematic (older format))
At the start: 8 parts

Commit message: Electronics - Misc. works
Continued (and checked board). All connections are probably OK.
Fixed hierarchical pins in APUs (affects all schematics)
Numbered elements for testing schematics
Parts:
- gave numbers to parts that had none: 8
Changed lines of the file:
@@
 $EndDescr
 $Comp
-L Connector:Screw_Terminal_01x10 J?
+L Connector:Screw_Terminal_01x10 J29
 U 1 1 5DC06D8D
 P 1600 1250
-F 0 "J?" H 1680 1242 50  0000 L CNN
+F 0 "J29" H 1680 1242 50  0000 L CNN
 F 1 "Screw_Terminal_01x10" H 1680 1151 50  0000 L CNN
 F 2 "" H 1600 1250 50  0001 C CNN
@@
 SDA
 $Comp
-L NXP:PCF8575 U?
+L NXP:PCF8575 U32
 U 1 1 5DC072AD
 P 4300 1050
-F 0 "U?" H 4300 1407 50  0000 C CNN
+F 0 "U32" H 4300 1407 50  0000 C CNN
 F 1 "PCF8575" H 4300 1316 50  0000 C CNN
 F 2 "IPC7351-Nominal:SOP65P775X200-24" H 4300 -650 50  0001 C CNN
@@
 $EndComp
 $Comp
-L Device:C_Small C?
+L Device:C_Small C40
 U 1 1 5DC072B4
 P 3700 1050
-F 0 "C?" V 3929 1050 50  0000 C CNN
+F 0 "C40" V 3929 1050 50  0000 C CNN
 F 1 "0.1u" V 3838 1050 50  0000 C CNN
 F 2 "" H 3700 1050 50  0001 C CNN
@@
 $EndComp
 $Comp
-L power:+3.3V #PWR?
+L power:+3.3V #PWR0271
 U 1 1 5DC072BB
 P 3800 1050
-F 0 "#PWR?" H 3800 900 50  0001 C CNN
+F 0 "#PWR0271" H 3800 900 50  0001 C CNN
 F 1 "+3.3V" V 3815 1178 50  0000 L CNN
 F 2 "" H 3800 1050 50  0001 C CNN
@@
 Connection ~ 3800 1050
 $Comp
-L power:GND #PWR?
+L power:GND #PWR0272
 U 1 1 5DC072C2
 P 3600 1050
-F 0 "#PWR?" H 3600 800 50  0001 C CNN
+F 0 "#PWR0272" H 3600 800 50  0001 C CNN
 F 1 "GND" V 3605 922 50  0000 R CNN
 F 2 "" H 3600 1050 50  0001 C CNN
@@
 $EndComp
 $Comp
-L power:GND #PWR?
+L power:GND #PWR0273
 U 1 1 5DC072C8
 P 3800 2550
-F 0 "#PWR?" H 3800 2300 50  0001 C CNN
+F 0 "#PWR0273" H 3800 2300 50  0001 C CNN
 F 1 "GND" V 3805 2422 50  0000 R CNN
 F 2 "" H 3800 2550 50  0001 C CNN
@@
 INT
 $Comp
-L power:GND #PWR?
+L power:GND #PWR0274
 U 1 1 5DC072CF
 P 3800 1250
-F 0 "#PWR?" H 3800 1000 50  0001 C CNN
+F 0 "#PWR0274" H 3800 1000 50  0001 C CNN
 F 1 "GND" V 3805 1122 50  0000 R CNN
 F 2 "" H 3800 1250 50  0001 C CNN
@@
 $EndComp
 $Comp
-L power:GND #PWR?
+L power:GND #PWR0275
 U 1 1 5DC072D5
 P 3800 1350
-F 0 "#PWR?" H 3800 1100 50  0001 C CNN
+F 0 "#PWR0275" H 3800 1100 50  0001 C CNN
 F 1 "GND" V 3805 1222 50  0000 R CNN
 F 2 "" H 3800 1350 50  0001 C CNN
@@
 $EndComp
 $Comp
-L power:GND #PWR?
+L power:GND #PWR0276
 U 1 1 5DC072DB
 P 3800 1450
-F 0 "#PWR?" H 3800 1200 50  0001 C CNN
+F 0 "#PWR0276" H 3800 1200 50  0001 C CNN
 F 1 "GND" V 3805 1322 50  0000 R CNN
 F 2 "" H 3800 1450 50  0001 C CNN
@@
 P 6500 1550
 AR Path="/5DB5DCD1/5DBEE2D9" Ref="U?"  Part="1"
-AR Path="/5DBF6FEB/5DBEE2D9" Ref="U?"  Part="1"
-F 0 "U?" H 6550 2228 50  0000 C CNN
+AR Path="/5DBF6FEB/5DBEE2D9" Ref="U33"  Part="1"
+F 0 "U33" H 6550 2228 50  0000 C CNN
 F 1 "74HC4051" H 6550 2137 50  0000 C CNN
 F 2 "" H 6500 1150 50  0001 C CNN
@@
 P 6550 2150
 AR Path="/5DB5DCD1/5DBEE2E9" Ref="#PWR?"  Part="1"
-AR Path="/5DBF6FEB/5DBEE2E9" Ref="#PWR?"  Part="1"
-F 0 "#PWR?" H 6550 1900 50  0001 C CNN
+AR Path="/5DBF6FEB/5DBEE2E9" Ref="#PWR0277"  Part="1"
+F 0 "#PWR0277" H 6550 1900 50  0001 C CNN
 F 1 "GND" H 6555 1977 50  0000 C CNN
 F 2 "" H 6550 2150 50  0001 C CNN
@@
 P 6950 1050
 AR Path="/5DB5DCD1/5DBEE2F1" Ref="C?"  Part="1"
-AR Path="/5DBF6FEB/5DBEE2F1" Ref="C?"  Part="1"
-F 0 "C?" V 7179 1050 50  0000 C CNN
+AR Path="/5DBF6FEB/5DBEE2F1" Ref="C41"  Part="1"
+F 0 "C41" V 7179 1050 50  0000 C CNN
 F 1 "0.1u" V 7088 1050 50  0000 C CNN
 F 2 "" H 6950 1050 50  0001 C CNN
@@
 P 7050 1050
 AR Path="/5DB5DCD1/5DBEE2F9" Ref="#PWR?"  Part="1"
-AR Path="/5DBF6FEB/5DBEE2F9" Ref="#PWR?"  Part="1"
-F 0 "#PWR?" H 7050 800 50  0001 C CNN
+AR Path="/5DBF6FEB/5DBEE2F9" Ref="#PWR0278"  Part="1"
+F 0 "#PWR0278" H 7050 800 50  0001 C CNN
 F 1 "GND" V 7055 922 50  0000 R CNN
 F 2 "" H 7050 1050 50  0001 C CNN
@@
 P 6300 1050
 AR Path="/5DB5DCD1/5DBEE2FF" Ref="#PWR?"  Part="1"
-AR Path="/5DBF6FEB/5DBEE2FF" Ref="#PWR?"  Part="1"
-F 0 "#PWR?" H 6300 900 50  0001 C CNN
+AR Path="/5DBF6FEB/5DBEE2FF" Ref="#PWR0279"  Part="1"
+F 0 "#PWR0279" H 6300 900 50  0001 C CNN
 F 1 "+3.3V" V 6315 1178 50  0000 L CNN
 F 2 "" H 6300 1050 50  0001 C CNN
@@
 AR Path="/5DBEE708" Ref="U?"  Part="1"
 AR Path="/5DB5DCD1/5DBEE708" Ref="U?"  Part="1"
-AR Path="/5DBF6FEB/5DBEE708" Ref="U?"  Part="1"
-F 0 "U?" H 2850 4897 60  0000 C CNN
+AR Path="/5DBF6FEB/5DBEE708" Ref="U31"  Part="1"
+F 0 "U31" H 2850 4897 60  0000 C CNN
 F 1 "74HC165" H 2850 4791 60  0000 C CNN
 F 2 "" H 5040 2780 60  0001 C CNN
@@
 $EndComp
 $Comp
-L power:GND #PWR?
+L power:GND #PWR0280
 U 1 1 5DBEE70F
 P 2250 4500
-F 0 "#PWR?" H 2250 4250 50  0001 C CNN
+F 0 "#PWR0280" H 2250 4250 50  0001 C CNN
 F 1 "GND" V 2255 4372 50  0000 R CNN
 F 2 "" H 2250 4500 50  0001 C CNN
@@
 $EndComp
 $Comp
-L power:GND #PWR?
+L power:GND #PWR0281
 U 1 1 5DBEE715
 P 3450 4650
-F 0 "#PWR?" H 3450 4400 50  0001 C CNN
+F 0 "#PWR0281" H 3450 4400 50  0001 C CNN
 F 1 "GND" V 3455 4522 50  0000 R CNN
 F 2 "" H 3450 4650 50  0001 C CNN
@@
 OSR_LATCH
 $Comp
-L Device:C_Small C?
+L Device:C_Small C39
 U 1 1 5DBEE720
 P 3450 3450
-F 0 "C?" H 3542 3496 50  0000 L CNN
+F 0 "C39" H 3542 3496 50  0000 L CNN
 F 1 "0.1u" H 3542 3405 50  0000 L CNN
 F 2 "" H 3450 3450 50  0001 C CNN
@@
 $EndComp
 $Comp
-L power:GND #PWR?
+L power:GND #PWR0282
 U 1 1 5DBEE727
 P 3450 3550
-F 0 "#PWR?" H 3450 3300 50  0001 C CNN
+F 0 "#PWR0282" H 3450 3300 50  0001 C CNN
 F 1 "GND" H 3455 3377 50  0000 C CNN
 F 2 "" H 3450 3550 50  0001 C CNN
@@
 	3450 3350 3650 3350
 $Comp
-L power:+3.3V #PWR?
+L power:+3.3V #PWR0283
 U 1 1 5DBEE72E
 P 3650 3350
-F 0 "#PWR?" H 3650 3200 50  0001 C CNN
+F 0 "#PWR0283" H 3650 3200 50  0001 C CNN
 F 1 "+3.3V" V 3665 3478 50  0000 L CNN
 F 2 "" H 3650 3350 50  0001 C CNN
@@
 $EndComp
 $Comp
-L Device:R_Network08 RN?
+L Device:R_Network08 RN14
 U 1 1 5DBEE734
 P 1350 3800
-F 0 "RN?" V 1867 3800 50  0000 C CNN
+F 0 "RN14" V 1867 3800 50  0000 C CNN
 F 1 "R_Network08" V 1776 3800 50  0000 C CNN
 F 2 "Resistor_THT:R_Array_SIP9" V 1825 3800 50  0001 C CNN
@@
 	1550 4200 2250 4200
 $Comp
-L power:+3.3V #PWR?
+L power:+3.3V #PWR0284
 U 1 1 5DBEE743
 P 1050 4200
-F 0 "#PWR?" H 1050 4050 50  0001 C CNN
+F 0 "#PWR0284" H 1050 4050 50  0001 C CNN
 F 1 "+3.3V" V 1065 4328 50  0000 L CNN
 F 2 "" H 1050 4200 50  0001 C CNN

Commit message: Electronics - Misc works
Parts:
- added BAR?: HDSP-4832_2, Display:HDSP-4832, symbol LED:HDSP-4832_2
- added C?: 0.1u, symbol Device:C_Small
- added RN?: R_Network08, Resistor_THT:R_Array_SIP9, symbol Device:R_Network08
- added U?: LM3914, symbol adessein:LM3914
- added U?: 74HC165, symbol pkl_misc:74HC165
- added U?: L7805, symbol Regulator_Linear:L7805
Connections:
- net labels added: LAND_LIGHT_LH, LAND_LIGHT_RH, LH_WING_DN, PARK_BREAK, RH_WING_DN, RUD_TRIM_CLK, RUD_TRIM_DT, TAXI_LIGHT
- net labels removed: ???_LIGHT, ??_LIGHT_LH, ??_LIGHT_RH, WXO_RH_NORM
- wire segments 16 -> 30
- no-connect marks 1 -> 2
Changed lines of the file:
@@
 EESchema Schematic File Version 4
 LIBS:CitationX_cockpit-cache
-EELAYER 26 0
+EELAYER 30 0
 EELAYER END
 $Descr A3 11693 16535 portrait
@@
 Wire Wire Line
 	3450 4200 3900 4200
-Text HLabel 4850 4000 0    50   Input ~ 0
+Text HLabel 5100 3750 0    50   Input ~ 0
 OSR_LATCH
 $Comp
@@
 GND_IDLE_HIGH
 Text Label 2250 3900 2    50   ~ 0
-???_LIGHT
+TAXI_LIGHT
 Text Label 2250 4000 2    50   ~ 0
-??_LIGHT_LH
+LAND_LIGHT_LH
 Text Label 2250 4100 2    50   ~ 0
-??_LIGHT_RH
+LAND_LIGHT_RH
 Text Label 2250 4200 2    50   ~ 0
-WXO_RH_NORM
+LH_WING_DN
+Text Label 4800 2450 0    50   ~ 0
+RUD_TRIM_CLK
+Text Label 4800 2550 0    50   ~ 0
+RUD_TRIM_DT
+$Comp
+L LED:HDSP-4832_2 BAR?
+U 1 1 5DE317D1
+P 6750 4000
+F 0 "BAR?" H 6750 3233 50  0000 C CNN
+F 1 "HDSP-4832_2" H 6750 3324 50  0000 C CNN
+F 2 "Display:HDSP-4832" H 6750 3200 50  0001 C CNN
+F 3 "https://docs.broadcom.com/docs/AV02-1798EN" H 4750 4200 50  0001 C CNN
+	1    6750 4000
+	-1   0    0    1
+$EndComp
+$Comp
+L adessein:LM3914 U?
+U 1 1 5DE51E4E
+P 5950 3250
+F 0 "U?" H 5950 3265 50  0000 C CNN
+F 1 "LM3914" H 5950 3174 50  0000 C CNN
+F 2 "" H 5950 3250 50  0001 C CNN
+F 3 "https://datasheet.lcsc.com/szlcsc/LM3914N-1-NOPB_C9408.pdf" H 5950 3250 50  0001 C CNN
+	1    5950 3250
+	1    0    0    -1
+$EndComp
+Text HLabel 2250 6450 0    50   Input ~ 0
+ISR_LATCH
+$Comp
+L pkl_misc:74HC165 U?
+U 1 1 5DE562A1
+P 2850 5850
+AR Path="/5DE562A1" Ref="U?"  Part="1"
+AR Path="/5DB5DCD1/5DE562A1" Ref="U?"  Part="1"
+AR Path="/5DBF6FEB/5DE562A1" Ref="U?"  Part="1"
+F 0 "U?" H 2850 6747 60  0000 C CNN
+F 1 "74HC165" H 2850 6641 60  0000 C CNN
+F 2 "" H 5040 4630 60  0001 C CNN
+F 3 "" H 5040 4630 60  0001 C CNN
+	1    2850 5850
+	1    0    0    -1
+$EndComp
+$Comp
+L power:GND #PWR?
+U 1 1 5DE562A7
+P 2250 6350
+F 0 "#PWR?" H 2250 6100 50  0001 C CNN
+F 1 "GND" V 2255 6222 50  0000 R CNN
+F 2 "" H 2250 6350 50  0001 C CNN
+F 3 "" H 2250 6350 50  0001 C CNN
+	1    2250 6350
+	0    1    1    0
+$EndComp
+$Comp
+L power:GND #PWR?
+U 1 1 5DE562AD
+P 3450 6500
+F 0 "#PWR?" H 3450 6250 50  0001 C CNN
+F 1 "GND" V 3455 6372 50  0000 R CNN
+F 2 "" H 3450 6500 50  0001 C CNN
+F 3 "" H 3450 6500 50  0001 C CNN
+	1    3450 6500
+	0    -1   -1   0
+$EndComp
+Text HLabel 2250 6250 0    50   Input ~ 0
+CLK
+NoConn ~ 3450 6250
+Wire Wire Line
+	3900 6050 3900 6750
+Wire Wire Line
+	3450 6050 3900 6050
+$Comp
+L Device:C_Small C?
+U 1 1 5DE562B7
+P 3450 5300
+F 0 "C?" H 3542 5346 50  0000 L CNN
+F 1 "0.1u" H 3542 5255 50  0000 L CNN
+F 2 "" H 3450 5300 50  0001 C CNN
+F 3 "~" H 3450 5300 50  0001 C CNN
+	1    3450 5300
+	1    0    0    -1
+$EndComp
+$Comp
+L power:GND #PWR?
+U 1 1 5DE562BD
+P 3450 5400
+F 0 "#PWR?" H 3450 5150 50  0001 C CNN
+F 1 "GND" H 3455 5227 50  0000 C CNN
+F 2 "" H 3450 5400 50  0001 C CNN
+F 3 "" H 3450 5400 50  0001 C CNN
+	1    3450 5400
+	1    0    0    -1
+$EndComp
+Wire Wire Line
+	3450 5200 3650 5200
+$Comp
+L power:+3.3V #PWR?
+U 1 1 5DE562C4
+P 3650 5200
+F 0 "#PWR?" H 3650 5050 50  0001 C CNN
+F 1 "+3.3V" V 3665 5328 50  0000 L CNN
+F 2 "" H 3650 5200 50  0001 C CNN
+F 3 "" H 3650 5200 50  0001 C CNN
+	1    3650 5200
+	0    1    1    0
+$EndComp
+$Comp
+L Device:R_Network08 RN?
+U 1 1 5DE562CA
+P 1350 5650
+F 0 "RN?" V 1867 5650 50  0000 C CNN
+F 1 "R_Network08" V 1776 5650 50  0000 C CNN
+F 2 "Resistor_THT:R_Array_SIP9" V 1825 5650 50  0001 C CNN
+F 3 "http://www.vishay.com/docs/31509/csc.pdf" H 1350 5650 50  0001 C CNN
+	1    1350 5650
+	0    -1   -1   0
+$EndComp
+Wire Wire Line
+	1550 5350 2250 5350
+Wire Wire Line
+	1550 5450 2250 5450
+Wire Wire Line
+	1550 5550 2250 5550
+Wire Wire Line
+	1550 5650 2250 5650
+Wire Wire Line
+	1550 5750 2250 5750
+Wire Wire Line
+	1550 5850 2250 5850
+Wire Wire Line
+	1550 5950 2250 5950
+Wire Wire Line
+	1550 6050 2250 6050
+$Comp
+L power:+3.3V #PWR?
+U 1 1 5DE562D8
+P 1050 6050
+F 0 "#PWR?" H 1050 5900 50  0001 C CNN
+F 1 "+3.3V" V 1065 6178 50  0000 L CNN
+F 2 "" H 1050 6050 50  0001 C CNN
+F 3 "" H 1050 6050 50  0001 C CNN
+	1    1050 6050
+	0    -1   -1   0
+$EndComp
+Text Label 2250 5450 2    50   ~ 0
+PARK_BREAK
+Wire Wire Line
+	1150 6050 1050 6050
+Wire Wire Line
+	3900 4900 2250 4900
+Wire Wire Line
+	2250 4900 2250 5250
+Text Label 2250 5350 2    50   ~ 0
+RH_WING_DN
+$Comp
+L Regulator_Linear:L7805 U?
+U 1 1 5DE57A12
+P 8750 2450
+F 0 "U?" H 8750 2692 50  0000 C CNN
+F 1 "L7805" H 8750 2601 50  0000 C CNN
+F 2 "" H 8775 2300 50  0001 L CIN
+F 3 "http://www.st.com/content/ccc/resource/technical/document/datasheet/41/4f/b3/b0/12/d4/47/88/CD00000444.pdf/files/CD00000444.pdf/jcr:content/translations/en.CD00000444.pdf" H 8750 2400 50  0001 C CNN
+	1    8750 2450
+	1    0    0    -1
+$EndComp
 $EndSCHEMATC

Commit message: Electronics - Added LED bar on pedestral
Parts:
- removed U?: LM3914, symbol adessein:LM3914
- removed U?: L7805, symbol Regulator_Linear:L7805
- added BAR? (x3): HDSP-4832_2, Display:HDSP-4832, symbol LED:HDSP-4832_2
- added C? (x5): 0.1u, symbol Device:C_Small
- added U? (x5): ULN2803A, symbol Transistor_Array:ULN2803A
- added U? (x5): 74HC595, symbol 74xx:74HC595
Connections:
- net labels added: +5V, OSR_IN, OSR_OUT
- wire segments 30 -> 196
Other:
- note added: "The LED bars are used for the trim and rudder position display"
- moved on the sheet: BAR?
