File: Electronics/Mainbord/board.sch (KiCad schematic (older format))
At the start: 51 parts, among them J16 Screw_Terminal_01x10, J17 Screw_Terminal_01x10, J18 Screw_Terminal_01x10, J19 Screw_Terminal_01x10, J20 Screw_Terminal_01x10, J21 Screw_Terminal_01x10, J22 Screw_Terminal_01x10, J23 Screw_Terminal_01x10, J24 Screw_Terminal_01x10, J25 Screw_Terminal_01x10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

Commit message: Electronics - Adds LCSC part numbers and footprints
Parts:
- U16, U18, U19: footprint IPC7351-Nominal:SOP65P775X200-24 -> Package_SO:SSOP-24_5.3x8.2mm_P0.65mm; LCSC (none) -> C12251
- U20: footprint (none) -> Package_SO:SOIC-16_3.9x9.9mm_P1.27mm; LCSC (none) -> C5947
- U21, U22: footprint (none) -> Package_SO:HTSSOP-16-1EP_4.4x5mm_P0.65mm_EP3.4x5mm; LCSC (none) -> C5645
- U23, U24, U25, U26, U27, U28, U29, U30: footprint (none) -> Package_SO:SOIC-16_3.9x9.9mm_P1.27mm; LCSC (none) -> C5613
Changed lines of the file:
@@
 F 0 "U17" H 2850 3087 60  0000 C CNN
 F 1 "ProMicro" H 2850 2981 60  0000 C CNN
-F 2 "" H 2950 1000 60  0000 C CNN
+F 2 "" H 2950 1000 60  0001 C CNN
 F 3 "" H 2950 1000 60  0000 C CNN
 	1    2850 2050
@@
 F 0 "U21" H 4750 2428 50  0000 C CNN
 F 1 "74HC4051" H 4750 2337 50  0000 C CNN
-F 2 "" H 4700 1350 50  0001 C CNN
+F 2 "Package_SO:HTSSOP-16-1EP_4.4x5mm_P0.65mm_EP3.4x5mm" H 4700 1350 50  0001 C CNN
 F 3 "http://www.ti.com/lit/ds/symlink/cd74hc4051.pdf" H 4700 1350 50  0001 C CNN
+F 4 " C5645" H 4700 1750 50  0001 C CNN "LCSC"
 	1    4700 1750
 	1    0    0    -1
@@
 F 0 "U22" H 6250 2428 50  0000 C CNN
 F 1 "74HC4051" H 6250 2337 50  0000 C CNN
-F 2 "" H 6200 1350 50  0001 C CNN
+F 2 "Package_SO:HTSSOP-16-1EP_4.4x5mm_P0.65mm_EP3.4x5mm" H 6200 1350 50  0001 C CNN
 F 3 "http://www.ti.com/lit/ds/symlink/cd74hc4051.pdf" H 6200 1350 50  0001 C CNN
+F 4 " C5645" H 6200 1750 50  0001 C CNN "LCSC"
 	1    6200 1750
 	1    0    0    -1
@@
 F 0 "U16" H 1450 4357 50  0000 C CNN
 F 1 "PCF8575" H 1450 4266 50  0000 C CNN
-F 2 "IPC7351-Nominal:SOP65P775X200-24" H 1450 2300 50  0001 C CNN
+F 2 "Package_SO:SSOP-24_5.3x8.2mm_P0.65mm" H 1450 2300 50  0001 C CNN
 F 3 "http://www.nxp.com/documents/data_sheet/PCF8575.pdf" H 1450 2200 50  0001 C CNN
 F 4 "NXP" H 1450 2000 50  0001 C CNN "Manuf"
@@
 F 6 "NXP PCF8575TS/1,112" H 1450 2100 50  0001 C CNN "BOM"
 F 7 "0x40" H 1450 4175 50  0000 C CNN "I2C adress"
+F 8 " C12251" H 1450 4000 50  0001 C CNN "LCSC"
 	1    1450 4000
 	1    0    0    -1
@@
 F 0 "U23" H 6450 5397 60  0000 C CNN
 F 1 "74HC165" H 6450 5291 60  0000 C CNN
-F 2 "" H 8640 3280 60  0001 C CNN
+F 2 "Package_SO:SOIC-16_3.9x9.9mm_P1.27mm" H 8640 3280 60  0001 C CNN
 F 3 "" H 8640 3280 60  0001 C CNN
+F 4 "C5613" H 6450 4500 50  0001 C CNN "LCSC"
 	1    6450 4500
 	1    0    0    -1
@@
 F 0 "U24" H 6450 7097 60  0000 C CNN
 F 1 "74HC165" H 6450 6991 60  0000 C CNN
-F 2 "" H 8640 4980 60  0001 C CNN
+F 2 "Package_SO:SOIC-16_3.9x9.9mm_P1.27mm" H 8640 4980 60  0001 C CNN
 F 3 "" H 8640 4980 60  0001 C CNN
+F 4 "C5613" H 6450 6200 50  0001 C CNN "LCSC"
 	1    6450 6200
 	1    0    0    -1
@@
 F 0 "U25" H 6450 8797 60  0000 C CNN
 F 1 "74HC165" H 6450 8691 60  0000 C CNN
-F 2 "" H 8640 6680 60  0001 C CNN
+F 2 "Package_SO:SOIC-16_3.9x9.9mm_P1.27mm" H 8640 6680 60  0001 C CNN
 F 3 "" H 8640 6680 60  0001 C CNN
+F 4 "C5613" H 6450 7900 50  0001 C CNN "LCSC"
 	1    6450 7900
 	1    0    0    -1
@@
 F 0 "U26" H 6450 10497 60  0000 C CNN
 F 1 "74HC165" H 6450 10391 60  0000 C CNN
-F 2 "" H 8640 8380 60  0001 C CNN
+F 2 "Package_SO:SOIC-16_3.9x9.9mm_P1.27mm" H 8640 8380 60  0001 C CNN
 F 3 "" H 8640 8380 60  0001 C CNN
+F 4 "C5613" H 6450 9600 50  0001 C CNN "LCSC"
 	1    6450 9600
 	1    0    0    -1
@@
 F 0 "U27" H 6450 12197 60  0000 C CNN
 F 1 "74HC165" H 6450 12091 60  0000 C CNN
-F 2 "" H 8640 10080 60  0001 C CNN
+F 2 "Package_SO:SOIC-16_3.9x9.9mm_P1.27mm" H 8640 10080 60  0001 C CNN
 F 3 "" H 8640 10080 60  0001 C CNN
+F 4 "C5613" H 6450 11300 50  0001 C CNN "LCSC"
 	1    6450 11300
 	1    0    0    -1
@@
 F 0 "U19" H 3500 4407 50  0000 C CNN
 F 1 "PCF8575" H 3500 4316 50  0000 C CNN
-F 2 "IPC7351-Nominal:SOP65P775X200-24" H 3500 2350 50  0001 C CNN
+F 2 "Package_SO:SSOP-24_5.3x8.2mm_P0.65mm" H 3500 2350 50  0001 C CNN
 F 3 "http://www.nxp.com/documents/data_sheet/PCF8575.pdf" H 3500 2250 50  0001 C CNN
 F 4 "NXP" H 3500 2050 50  0001 C CNN "Manuf"
@@
 F 6 "NXP PCF8575TS/1,112" H 3500 2150 50  0001 C CNN "BOM"
 F 7 "0x41" H 3500 4225 50  0000 C CNN "I2C adress"
+F 8 " C12251" H 3500 4050 50  0001 C CNN "LCSC"
 	1    3500 4050
 	1    0    0    -1
@@
 F 0 "U20" H 3500 9628 50  0000 C CNN
 F 1 "74HC595" H 3500 9537 50  0000 C CNN
-F 2 "" H 3500 8850 50  0001 C CNN
+F 2 "Package_SO:SOIC-16_3.9x9.9mm_P1.27mm" H 3500 8850 50  0001 C CNN
 F 3 "http://www.ti.com/lit/ds/symlink/sn74hc595.pdf" H 3500 8850 50  0001 C CNN
+F 4 "C5947" H 3500 8850 50  0001 C CNN "LCSC"
 	1    3500 8850
 	1    0    0    -1
@@
 F 0 "U28" H 6450 14097 60  0000 C CNN
 F 1 "74HC165" H 6450 13991 60  0000 C CNN
-F 2 "" H 8640 11980 60  0001 C CNN
+F 2 "Package_SO:SOIC-16_3.9x9.9mm_P1.27mm" H 8640 11980 60  0001 C CNN
 F 3 "" H 8640 11980 60  0001 C CNN
+F 4 "C5613" H 6450 13200 50  0001 C CNN "LCSC"
 	1    6450 13200
 	1    0    0    -1
@@
 F 0 "U29" H 9900 5397 60  0000 C CNN
 F 1 "74HC165" H 9900 5291 60  0000 C CNN
-F 2 "" H 12090 3280 60  0001 C CNN
+F 2 "Package_SO:SOIC-16_3.9x9.9mm_P1.27mm" H 12090 3280 60  0001 C CNN
 F 3 "" H 12090 3280 60  0001 C CNN
+F 4 "C5613" H 9900 4500 50  0001 C CNN "LCSC"
 	1    9900 4500
 	1    0    0    -1
@@
 F 0 "U30" H 9900 7097 60  0000 C CNN
 F 1 "74HC165" H 9900 6991 60  0000 C CNN
-F 2 "" H 12090 4980 60  0001 C CNN
+F 2 "Package_SO:SOIC-16_3.9x9.9mm_P1.27mm" H 12090 4980 60  0001 C CNN
 F 3 "" H 12090 4980 60  0001 C CNN
+F 4 "C5613" H 9900 6200 50  0001 C CNN "LCSC"
 	1    9900 6200
 	1    0    0    -1
@@
 F 0 "U18" H 3450 6407 50  0000 C CNN
 F 1 "PCF8575" H 3450 6316 50  0000 C CNN
-F 2 "IPC7351-Nominal:SOP65P775X200-24" H 3450 4350 50  0001 C CNN
+F 2 "Package_SO:SSOP-24_5.3x8.2mm_P0.65mm" H 3450 4350 50  0001 C CNN
 F 3 "http://www.nxp.com/documents/data_sheet/PCF8575.pdf" H 3450 4250 50  0001 C CNN
 F 4 "NXP" H 3450 4050 50  0001 C CNN "Manuf"
@@
 F 6 "NXP PCF8575TS/1,112" H 3450 4150 50  0001 C CNN "BOM"
 F 7 "0x42" H 3450 6225 50  0000 C CNN "I2C adress"
+F 8 " C12251" H 3450 6050 50  0001 C CNN "LCSC"
 	1    3450 6050
 	1    0    0    -1
