File: Electronics/Pedestral/Pedestral.sch (KiCad schematic (older format))
At the start: 35 parts, among them J29 Screw_Terminal_01x10, U31 74HC165, U32 PCF8575, U33 74HC4051

Commit message: Electrnonics - Change label on pedestral after separation
Parts:
- added J?: Conn_02x08_Odd_Even, symbol Connector_Generic:Conn_02x08_Odd_Even
Connections:
- net ISR_IN is gone; now on net GND: U31.10 (SER)
- net +3V3: now also J?.2 (Pin_2)
- net +5V: now also U?.21 (VCC), J?.1 (Pin_1)
- net ADC: now also U?.12 (D9/A9)
- net CLK: now also U?.18 (A1)
- net GND: now also U?.23 (GND), J?.11 (Pin_11), J?.15 (Pin_15), J?.3 (Pin_3), J?.4 (Pin_4), J?.7 (Pin_7)
- net ISR_LATCH: now also U?.16 (D15/SCK)
- net ISR_OUT: now also U?.17 (A0)
- net OSR_IN: now also U?.20 (A3)
- net OSR_LATCH: now also U?.19 (A2)
- net RX: now also U?.2 (D0/RX), J?.5 (Pin_5); no longer U?.1 (D1/TX)
- net TX: now also U?.1 (D1/TX), J?.9 (Pin_9); no longer U?.2 (D0/RX)
- net RST: now reaches U?.22 (RST)
- net RST: now also J?.13 (Pin_13)
- net OSR_OUT: no longer names the net of U?.9 (QH')
Other:
- moved on the sheet: C40, C41, J29, U32, U33, U?

Commit message: Electronics - Misc works
Parts:
- added C?: 0.1u, symbol Device:C_Small
- added U?: WeMos_mini, symbol wemos_mini:WeMos_mini
- added U?: 74HC595, symbol 74xx:74HC595
Connections:
- wire segments 159 -> 170
Other:
- moved on the sheet: C41, U33

Commit message: Electronics - Footprints and LCSC for APU and Pedestral
Parts:
- removed U?: WeMos_mini, symbol wemos_mini:WeMos_mini
- U31, U?: footprint (none) -> Package_SO:SOIC-16_3.9x9.9mm_P1.27mm; LCSC (none) -> C5613
- U32: footprint IPC7351-Nominal:SOP65P775X200-24 -> Package_SO:SSOP-24_5.3x8.2mm_P0.65mm; LCSC (none) -> C12251
- U33: footprint (none) -> Package_SO:HTSSOP-16-1EP_4.4x5mm_P0.65mm_EP3.4x5mm; LCSC (none) -> C5645
- U? (x5): footprint (none) -> Package_SO:SOIC-18W_7.5x11.6mm_P1.27mm; LCSC (none) -> C9683
- U?: footprint (none) -> promicro:ProMicro
- U? (x6): footprint (none) -> Package_SO:SOIC-16_3.9x9.9mm_P1.27mm; LCSC (none) -> C5947
Changed lines of the file:
@@
 F 0 "U32" H 6900 1357 50  0000 C CNN
 F 1 "PCF8575" H 6900 1266 50  0000 C CNN
-F 2 "IPC7351-Nominal:SOP65P775X200-24" H 6900 -700 50  0001 C CNN
+F 2 "Package_SO:SSOP-24_5.3x8.2mm_P0.65mm" H 6900 -700 50  0001 C CNN
 F 3 "http://www.nxp.com/documents/data_sheet/PCF8575.pdf" H 6900 -800 50  0001 C CNN
 F 4 "NXP" H 6900 -1000 50  0001 C CNN "Manuf"
@@
 F 6 "NXP PCF8575TS/1,112" H 6900 -900 50  0001 C CNN "BOM"
 F 7 "0x40" H 6900 1175 50  0000 C CNN "I2C adress"
+F 8 "C12251" H 6900 1000 50  0001 C CNN "LCSC"
 	1    6900 1000
 	1    0    0    -1
@@
 AR Path="/5DB5DCD1/5DBEE2D9" Ref="U?"  Part="1"
 AR Path="/5DBF6FEB/5DBEE2D9" Ref="U33"  Part="1"
+AR Path="/5DBEE2D9" Ref="U33"  Part="1"
 F 0 "U33" H 12400 12628 50  0000 C CNN
 F 1 "74HC4051" H 12400 12537 50  0000 C CNN
-F 2 "" H 12350 11550 50  0001 C CNN
+F 2 "Package_SO:HTSSOP-16-1EP_4.4x5mm_P0.65mm_EP3.4x5mm" H 12350 11550 50  0001 C CNN
 F 3 "http://www.ti.com/lit/ds/symlink/cd74hc4051.pdf" H 12350 11550 50  0001 C CNN
+F 4 "C5645" H 12350 11950 50  0001 C CNN "LCSC"
 	1    12350 11950
 	1    0    0    -1
@@
 AR Path="/5DB5DCD1/5DBEE708" Ref="U?"  Part="1"
 AR Path="/5DBF6FEB/5DBEE708" Ref="U31"  Part="1"
-F 0 "U31" H 2850 4897 60  0000 C CNN
+F 0 "U?" H 2850 4897 60  0000 C CNN
 F 1 "74HC165" H 2850 4791 60  0000 C CNN
-F 2 "" H 5040 2780 60  0001 C CNN
+F 2 "Package_SO:SOIC-16_3.9x9.9mm_P1.27mm" H 5040 2780 60  0001 C CNN
 F 3 "" H 5040 2780 60  0001 C CNN
+F 4 "C5613" H 2850 4000 50  0001 C CNN "LCSC"
 	1    2850 4000
 	1    0    0    -1
@@
 F 0 "U?" H 2850 6747 60  0000 C CNN
 F 1 "74HC165" H 2850 6641 60  0000 C CNN
-F 2 "" H 5040 4630 60  0001 C CNN
+F 2 "Package_SO:SOIC-16_3.9x9.9mm_P1.27mm" H 5040 4630 60  0001 C CNN
 F 3 "" H 5040 4630 60  0001 C CNN
+F 4 "C5613" H 2850 5850 50  0001 C CNN "LCSC"
 	1    2850 5850
 	1    0    0    -1
@@
 F 0 "U?" H 11100 5067 50  0000 C CNN
 F 1 "ULN2803A" H 11100 4976 50  0000 C CNN
-F 2 "" H 11150 3850 50  0001 L CNN
+F 2 "Package_SO:SOIC-18W_7.5x11.6mm_P1.27mm" H 11150 3850 50  0001 L CNN
 F 3 "http://www.ti.com/lit/ds/symlink/uln2803a.pdf" H 11200 4300 50  0001 C CNN
+F 4 "C9683" H 11100 4500 50  0001 C CNN "LCSC"
 	1    11100 4500
 	1    0    0    -1
@@
 F 0 "U?" H 11100 6467 50  0000 C CNN
 F 1 "ULN2803A" H 11100 6376 50  0000 C CNN
-F 2 "" H 11150 5250 50  0001 L CNN
+F 2 "Package_SO:SOIC-18W_7.5x11.6mm_P1.27mm" H 11150 5250 50  0001 L CNN
 F 3 "http://www.ti.com/lit/ds/symlink/uln2803a.pdf" H 11200 5700 50  0001 C CNN
+F 4 "C9683" H 11100 5900 50  0001 C CNN "LCSC"
 	1    11100 5900
 	1    0    0    -1
@@
 F 0 "U?" H 11100 7867 50  0000 C CNN
 F 1 "ULN2803A" H 11100 7776 50  0000 C CNN
-F 2 "" H 11150 6650 50  0001 L CNN
+F 2 "Package_SO:SOIC-18W_7.5x11.6mm_P1.27mm" H 11150 6650 50  0001 L CNN
 F 3 "http://www.ti.com/lit/ds/symlink/uln2803a.pdf" H 11200 7100 50  0001 C CNN
+F 4 "C9683" H 11100 7300 50  0001 C CNN "LCSC"
 	1    11100 7300
 	1    0    0    -1
@@
 F 0 "U?" H 11100 9267 50  0000 C CNN
 F 1 "ULN2803A" H 11100 9176 50  0000 C CNN
-F 2 "" H 11150 8050 50  0001 L CNN
+F 2 "Package_SO:SOIC-18W_7.5x11.6mm_P1.27mm" H 11150 8050 50  0001 L CNN
 F 3 "http://www.ti.com/lit/ds/symlink/uln2803a.pdf" H 11200 8500 50  0001 C CNN
+F 4 "C9683" H 11100 8700 50  0001 C CNN "LCSC"
 	1    11100 8700
 	1    0    0    -1
@@
 F 0 "U?" H 11100 10667 50  0000 C CNN
 F 1 "ULN2803A" H 11100 10576 50  0000 C CNN
-F 2 "" H 11150 9450 50  0001 L CNN
+F 2 "Package_SO:SOIC-18W_7.5x11.6mm_P1.27mm" H 11150 9450 50  0001 L CNN
 F 3 "http://www.ti.com/lit/ds/symlink/uln2803a.pdf" H 11200 9900 50  0001 C CNN
+F 4 "C9683" H 11100 10100 50  0001 C CNN "LCSC"
 	1    11100 10100
 	1    0    0    -1
@@
 AR Path="/5DC174D4/5DFDCD39" Ref="U?"  Part="1"
 AR Path="/5DBF6FEB/5DFDCD39" Ref="U?"  Part="1"
+AR Path="/5DFDCD39" Ref="U?"  Part="1"
 F 0 "U?" H 9100 9678 50  0000 C CNN
 F 1 "74HC595" H 9100 9587 50  0000 C CNN
-F 2 "" H 9100 8900 50  0001 C CNN
+F 2 "Package_SO:SOIC-16_3.9x9.9mm_P1.27mm" H 9100 8900 50  0001 C CNN
 F 3 "http://www.ti.com/lit/ds/symlink/sn74hc595.pdf" H 9100 8900 50  0001 C CNN
+F 4 "C5947" H 9100 8900 50  0001 C CNN "LCSC"
 	1    9100 8900
 	1    0    0    -1
@@
 F 0 "U?" H 6600 5478 50  0000 C CNN
 F 1 "74HC595" H 6600 5387 50  0000 C CNN
-F 2 "" H 6600 4700 50  0001 C CNN
+F 2 "Package_SO:SOIC-16_3.9x9.9mm_P1.27mm" H 6600 4700 50  0001 C CNN
 F 3 "http://www.ti.com/lit/ds/symlink/sn74hc595.pdf" H 6600 4700 50  0001 C CNN
+F 4 "C5947" H 6600 4700 50  0001 C CNN "LCSC"
 	1    6600 4700
 	1    0    0    -1
@@
 AR Path="/5DC174D4/5E07F9BE" Ref="U?"  Part="1"
 AR Path="/5DBF6FEB/5E07F9BE" Ref="U?"  Part="1"
+AR Path="/5E07F9BE" Ref="U?"  Part="1"
 F 0 "U?" H 8300 8278 50  0000 C CNN
 F 1 "74HC595" H 8300 8187 50  0000 C CNN
-F 2 "" H 8300 7500 50  0001 C CNN
+F 2 "Package_SO:SOIC-16_3.9x9.9mm_P1.27mm" H 8300 7500 50  0001 C CNN
 F 3 "http://www.ti.com/lit/ds/symlink/sn74hc595.pdf" H 8300 7500 50  0001 C CNN
+F 4 "C5947" H 8300 7500 50  0001 C CNN "LCSC"
 	1    8300 7500
 	1    0    0    -1
@@
 AR Path="/5DC174D4/5E07F9EB" Ref="U?"  Part="1"
 AR Path="/5DBF6FEB/5E07F9EB" Ref="U?"  Part="1"
+AR Path="/5E07F9EB" Ref="U?"  Part="1"
 F 0 "U?" H 7450 6878 50  0000 C CNN
 F 1 "74HC595" H 7450 6787 50  0000 C CNN
-F 2 "" H 7450 6100 50  0001 C CNN
+F 2 "Package_SO:SOIC-16_3.9x9.9mm_P1.27mm" H 7450 6100 50  0001 C CNN
 F 3 "http://www.ti.com/lit/ds/symlink/sn74hc595.pdf" H 7450 6100 50  0001 C CNN
+F 4 "C5947" H 7450 6100 50  0001 C CNN "LCSC"
 	1    7450 6100
 	1    0    0    -1
@@
 F 0 "U?" H 9950 11078 50  0000 C CNN
 F 1 "74HC595" H 9950 10987 50  0000 C CNN
-F 2 "" H 9950 10300 50  0001 C CNN
+F 2 "Package_SO:SOIC-16_3.9x9.9mm_P1.27mm" H 9950 10300 50  0001 C CNN
 F 3 "http://www.ti.com/lit/ds/symlink/sn74hc595.pdf" H 9950 10300 50  0001 C CNN
+F 4 "C5947" H 9950 10300 50  0001 C CNN "LCSC"
 	1    9950 10300
 	1    0    0    -1
@@
 F 0 "U?" H 1750 2987 60  0000 C CNN
 F 1 "ProMicro" H 1750 2881 60  0000 C CNN
-F 2 "" H 1850 900 60  0000 C CNN
+F 2 "promicro:ProMicro" H 1850 900 60  0000 C CNN
 F 3 "" H 1850 900 60  0000 C CNN
 	1    1750 1950
@@
 CLK
 $Comp
-L wemos_mini:WeMos_mini U?
-U 1 1 5DE7632B
-P 1700 -650
-F 0 "U?" H 1700 -13 60  0000 C CNN
-F 1 "WeMos_mini" H 1700 -119 60  0000 C CNN
-F 2 "" H 2250 -1350 60  0000 C CNN
-F 3 "http://www.wemos.cc/Products/d1_mini.html" H 1700 -119 60  0001 C CNN
-	1    1700 -650
-	1    0    0    -1
-$EndComp
-$Comp
-L power:GND #PWR?
-U 1 1 5DF1ACF8
-P 1200 -900
-F 0 "#PWR?" H 1200 -1150 50  0001 C CNN
-F 1 "GND" V 1205 -1028 50  0000 R CNN
-F 2 "" H 1200 -900 50  0001 C CNN
-F 3 "" H 1200 -900 50  0001 C CNN
-	1    1200 -900
-	0    1    1    0
-$EndComp
-$Comp
-L power:+5V #PWR?
-U 1 1 5DF23FC9
-P 1200 -1000
-F 0 "#PWR?" H 1200 -1150 50  0001 C CNN
-F 1 "+5V" V 1215 -872 50  0000 L CNN
-F 2 "" H 1200 -1000 50  0001 C CNN
-F 3 "" H 1200 -1000 50  0001 C CNN
-	1    1200 -1000
-	0    -1   -1   0
-$EndComp
-Text Label 1200 -500 2    50   ~ 0
-SCL
-Text Label 1200 -600 2    50   ~ 0
-SDA
-Text Label 2200 -400 0    50   ~ 0
-ADC
-Text Label 2200 -500 0    50   ~ 0
-ISR_LATCH
-Text Label 2200 -600 0    50   ~ 0
-OSR_LATCH
-Text Label 2200 -700 0    50   ~ 0
-CLK
-Text Label 2200 -800 0    50   ~ 0
-OSR_IN
-Text Label 2200 -900 0    50   ~ 0
-ISR_OUT
-Text Label 1200 -700 2    50   ~ 0
-INT
-$Comp
 L Device:C_Small C?
 U 1 1 5DF41493
@@
 F 0 "U?" H 10800 13028 50  0000 C CNN
 F 1 "74HC595" H 10800 12937 50  0000 C CNN
-F 2 "" H 10800 12250 50  0001 C CNN
+F 2 "Package_SO:SOIC-16_3.9x9.9mm_P1.27mm" H 10800 12250 50  0001 C CNN
 F 3 "http://www.ti.com/lit/ds/symlink/sn74hc595.pdf" H 10800 12250 50  0001 C CNN
+F 4 "C5947" H 10800 12250 50  0001 C CNN "LCSC"
 	1    10800 12250
 	1    0    0    -1
@@
 Wire Wire Line
 	11200 12050 12050 12050
-Text Label 1200 -800 2    50   ~ 0
-ADC_E
 Wire Notes Line
 	5300 11100 12900 11100
